File: Programmable_Buck_Boost/Programmable_Buck_Boost/Programmable_Buck_Boost.kicad_sch (KiCad schematic)
At the start: 38 parts, among them J2 DC INPUT, Q5 IRF3205, Q6 IRF3205, Q7 2N7002, U4 TL494, U6 IR2101

Commit message: Finalize Schematic
Parts:
- removed TP3: TestPoint, symbol Connector:TestPoint
- added C1: C0603/1nF, Capacitor_SMD:C_0603_1608Metric, symbol Device:C
- added C10, C13, C14, C9: C0805/22uF, Capacitor_SMD:C_0603_1608Metric, symbol Device:C
- added C11, C4: C0603/0.1uF, Capacitor_SMD:C_0603_1608Metric, symbol Device:C
- added C12: Cp/10uF/100V, symbol Device:C_Polarized
- added C2, C5: C0603/100nF, Capacitor_SMD:C_0603_1608Metric, symbol Device:C
- added C22, C3, C7: C0603/1uF, Capacitor_SMD:C_0603_1608Metric, symbol Device:C
- added C6, C8: C0603/10uF, Capacitor_SMD:C_0603_1608Metric, symbol Device:C
- added D2, D3: SS34, Diode_SMD:D_SMA, symbol Diode:SS34
- added J1: Conn_01x05_Pin, symbol Connector:Conn_01x05_Pin
- added J3: Conn_01x03_Pin, symbol Connector:Conn_01x03_Pin
- added J4: Conn_01x04_Pin, symbol Connector:Conn_01x04_Pin
- added L1: 100uH, symbol Device:L
- added L2: 4.7uH, symbol Device:L
- added R1, R6: R0603/4.7K, Resistor_SMD:R_0603_1608Metric, symbol Device:R
- added R10, R11, R2, R4, R7, R8: R0603/100K, Resistor_SMD:R_0603_1608Metric, symbol Device:R
- added R3: R0603/51K, Resistor_SMD:R_0603_1608Metric, symbol Device:R
- added R5: R0603/56k, Resistor_SMD:R_0603_1608Metric, symbol Device:R
- added R9: R0603/0.82, Resistor_SMD:R_0603_1608Metric, symbol Device:R
- added SW1: RotaryEncoder_Switch, symbol Device:RotaryEncoder_Switch
- added U1: MP1470, Package_TO_SOT_SMD:TSOT-23-6, symbol Regulator_Switching:MP1470
- added U2: MSPS003F4SPW20R, Package_SO:TSSOP-20_4.4x6.5mm_P0.65mm, symbol Minh_Symbol:MSPS003F4SPW20R
- added U3: MCP601-xOT, Package_TO_SOT_SMD:SOT-23-5, symbol Amplifier_Operational:MCP601-xOT
- added U5: EG1198, Package_SO:HSOP-8-1EP_3.9x4.9mm_P1.27mm_EP2.3x2.3mm, symbol Minh_Symbol:EG1198
- C15, C16, C17, C18, C19, C21: footprint (none) -> Capacitor_SMD:C_0603_1608Metric
- C20: value 220uF -> 220uF/65V
- R36, R39, R40: value R0603/10k -> R0603/100k
- R37: value R0603/220R -> R0603/2.2K
- R53: value RS/0.5R -> RS/0.1R
- R55: value R0603/56k -> R0603/150K
- U4: footprint Package_DIP:CERDIP-16_W7.62mm_SideBrazed_LongPads -> Package_SO:SOIC-16_3.9x9.9mm_P1.27mm
Connections:
- net V_set is gone; now on net V_FB: R52.1, R55.1
- net +12V: now also C3.1, C4.1
- net +5V: now also U3.5 (V+)
- net GND: now also C1.2, C10.2, C12.2, C13.2, C14.2, C2.2, C22.2, C3.2, C4.2, C5.1, C5.2, C6.2, C8.2, C9.2, D2.2 (A), D3.2 (A), J1.2 (Pin_2), J3.3 (Pin_3), J4.1 (Pin_1), R11.2, R4.1, R8.2, SW1.S2, U1.1 (GND), U2.7 (VSS), U3.2 (V-), U5.2 (GND)
- net V_SET: now reaches C16.2, R39.1, R40.2, U4.2 (1IN-)
- net V_SET: now also R3.2, U3.1; no longer U4.15 (2IN-)
- net I_SET: now reaches C17.2, R36.1, R37.2
- net I_SET: now also U4.15 (2IN-), C6.1, R1.2
- net I_set renamed I_FB
- net V_fb renamed V_FB
- net V_FB: now also C1.1
- new net: C8.1, R6.2, U3.3 (+)
- new net: C9.1, L2.2, R7.2
- new net: C7.1, D3.1 (K), L2.1, U1.2 (SW)
- new net: C7.2, U1.6 (BST)
- new net: C13.1, C14.1, L1.2, R10.2
- new net: C11.1, D2.1 (K), L1.1, R9.1, U5.7 (VS)
- new net: C11.2, U5.6 (VB)
- new net: R3.1, R4.2, U3.4 (-)
- new net: R2.1, U1.5 (EN)
- new net: C10.1, R2.2, U1.3 (IN)
- new net: SW1.A, U2.20 (PA25/A2)
- new net: SW1.B, U2.19 (PA24/A3)
- new net: R9.2, U5.8 (IS)
- new net +3.3V: C2.1, C22.1, J1.1 (Pin_1), J4.2 (Pin_2), R5.1, SW1.C, U2.9 (VDD)
- new net 12VFB: R10.1, R11.1, U5.4 (FB)
- new net 3V3FB: R7.1, R8.1, U1.4 (FB)
- new net ENC_BUTTON: R5.2, SW1.S1, U2.18 (PA23)
- new net I2C0_SCL: J4.3 (Pin_3), U2.11 (PA0)
- new net I2C0_SDA: J4.4 (Pin_4), U2.12 (PA1)
- new net I_PWM: R1.1, U2.8 (PA2)
- new net NRST: J1.3 (Pin_3), U2.4 (NRST)
- new net SWCLK: J1.4 (Pin_4), U2.16 (PA20/A6/SWCLK)
- new net SWDIO: J1.5 (Pin_5), U2.15 (PA19/SWDIO)
- new net UART0_RX: J3.1 (Pin_1), U2.14 (PA18/A7)
- new net UART0_TX: J3.2 (Pin_2), U2.13 (PA17/A9)
- new net VIN: C12.1, U5.1 (VIN), U5.9 (VIN)
- new net VSETPOINT: R6.1
- no-connect marks 0 -> 1
Other:
- note added: "Vin: 0.2V-48V"
- note added: "Vin: 12V-70V"
- moved on the sheet: C15, C16, C17, C18, C19, C20, C21, D1, D8, D9, J2, L3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

Commit message: Add current sense circuit
Parts:
- removed C11: C0603/0.1uF, Capacitor_SMD:C_0603_1608Metric, symbol Device:C
- removed C22: C0603/1uF, Capacitor_SMD:C_0603_1608Metric, symbol Device:C
- removed J3: Conn_01x03_Pin, symbol Connector:Conn_01x03_Pin
- removed R36, R39: R0603/100k, Resistor_SMD:R_0603_1608Metric, symbol Device:R
- removed R45: R0603/4.7k, Resistor_SMD:R_0603_1608Metric, symbol Device:R
- removed U2: MSPS003F4SPW20R, Package_SO:TSSOP-20_4.4x6.5mm_P0.65mm, symbol Minh_Symbol:MSPS003F4SPW20R
- removed U5: EG1198, Package_SO:HSOP-8-1EP_3.9x4.9mm_P1.27mm_EP2.3x2.3mm, symbol Minh_Symbol:EG1198
- added C11, C22, C23: Cp/470uF/63V, Capacitor_THT:CP_Radial_D12.5mm_P5.00mm, symbol Device:C_Polarized
- added C24: C0603/1nF, Capacitor_SMD:C_0603_1608Metric, symbol Device:C
- added C25: C0603/100nF, Capacitor_SMD:C_0603_1608Metric, symbol Device:C
- added R12, R13, R14, R15: R0603/150K, Resistor_SMD:R_0603_1608Metric, symbol Device:R
- added R16: R0603/10K, Resistor_SMD:R_0603_1608Metric, symbol Device:R
- added U2: XL7005A, Package_SO:SOIC-8-1EP_3.9x4.9mm_P1.27mm_EP2.29x3mm, symbol Minh_Symbol:XL7005A
- added U5: STM32F103C8Tx, Package_QFP:LQFP-48_7x7mm_P0.5mm, symbol MCU_ST_STM32F1:STM32F103C8Tx
- added U7: MCP601-xOT, Package_TO_SOT_SMD:SOT-23-5, symbol Amplifier_Operational:MCP601-xOT
- C12: value Cp/10uF/100V -> Cp/47uF/63V; footprint (none) -> Capacitor_THT:CP_Radial_D8.0mm_P3.50mm
- C2: value C0603/100nF -> C0603/33nF
- C9: value C0805/22uF -> C0603/10uF
- D2: value SS34 -> SS24
- L1: value 100uH -> L/47uH /620mA; footprint (none) -> Inductor_SMD:L_Abracon_ASPI-0425
- L3: value 47uF -> 47uF/25A
- Q5, Q6: value IRF3205 -> IRFB4110PbF
- R10: value R0603/100K -> R0603/30K
- R11: value R0603/100K -> R0603/3.3K
- R37: value R0603/2.2K -> R0603/100K
- R53: value RS/0.1R -> RS/0.002R
- R7: value R0603/100K -> R0603/75K
- R8: value R0603/100K -> R0603/24K
- R9: value R0603/0.82 -> R0603/100K
Connections:
- net VIN is gone; now on net VCC: C12.1
- net +12V: now also C13.1, C14.1, C2.2, L1.2, R10.1, R44.2
- net +3.3V: now also C9.1, L2.2, R7.1, R16.1, U7.5 (V+); no longer C2.1
- net +5V: no longer R44.2
- net 12VFB: now also C2.1, R10.2, U2.3 (FB); no longer R10.1
- net 3V3FB: now also R7.2; no longer R7.1
- net GND: now also C11.2, C22.2, C23.2, C25.2, R13.1, U2.5 (GND), U2.6 (GND), U2.7 (GND), U2.8 (GND), U2.9 (GND), U7.2 (V-); no longer C2.2
- net I_FB: now also C25.1, R15.2; no longer C20.2, C21.2, R53.2
- net VCC: now also R9.1, C11.1, C22.1, C23.1, U2.1 (VIN)
- net at U4.10 (E2), U4.9 (E1): now also Q7.1 (G), R46.2, R47.1, U6.2 (HIN)
- net at D2.1 (K), L1.1: now also U2.2 (SW); no longer R9.1
- net at R9.2: now also U2.4 (EN)
- new net: C20.2, C21.2, R12.1, R53.2
- new net: C24.1, R14.2, R15.1, U7.1
- new net: U5.23 (VSS), U5.35 (VSS), U5.47 (VSS)
- new net: R16.2, U5.7 (NRST)
- new net: C24.2, R13.2, R14.1, U7.4 (-)
- new net: R12.2, U7.3 (+)
- no-connect marks 1 -> 0
Other:
- note added: "75kHz"
- note added: "Iout:0.01-20A"
- note added: "Vin: 12V-50V"
- note added: "Vout: 0.2V-48V"
- note removed: "100mV"
- note removed: "5V logic"
- note removed: "PWM<90%"
- note removed: "Vin: 0.2V-48V"
- note removed: "Vin: 12V-70V"
- note removed: "~100kHz"
- moved on the sheet: C1, C10, C12, C13, C14, C15, C16, C17, C18, C19, C20, C21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

Commit message: Change design
Parts:
- added C26, C27, C28, C29, C30, C31: C0603/100nF, Capacitor_SMD:C_0603_1608Metric, symbol Device:C
- added J3: DC OUTPUT, TerminalBlock_Phoenix:TerminalBlock_Phoenix_MKDS-1,5-2-5.08_1x02_P5.08mm_Horizontal, symbol Connector:Screw_Terminal_01x02
- added R17: R0603/10K, Resistor_SMD:R_0603_1608Metric, symbol Device:R
- added R18, R19: R0603/100K, Resistor_SMD:R_0603_1608Metric, symbol Device:R
- C20, J1: footprint (none) -> Connector_JST:JST_XH_B5B-XH-AM_1x05_P2.50mm_Vertical
- J4: footprint (none) -> Connector_PinSocket_2.54mm:PinSocket_1x04_P2.54mm_Vertical
- SW1: footprint (none) -> Rotary_Encoder:RotaryEncoder_Alps_EC11E-Switch_Vertical_H20mm
Connections:
- net VSETPOINT is gone; now on net V_PWM: R6.1
- net +12V: now also C10.1, R2.2, U1.3 (IN)
- net +3.3V: now also U5.1 (VBAT), U5.24 (VDD), U5.36 (VDD), U5.48 (VDD), U5.9 (VDDA), C26.1, C27.1, C28.1, C29.1, C31.1
- net ENC_BUTTON: now also U5.19 (PB1)
- net GND: now also U5.23 (VSS), U5.35 (VSS), U5.47 (VSS), U5.8 (VSSA), C26.2, C27.2, C28.2, C29.2, C30.1, C31.2, R17.2, R18.2, R19.2
- net I_FB: now also U5.10 (PA0), R18.1
- net I_PWM: now also U5.39 (PB3)
- net NRST: now also R16.2, U5.7 (NRST), C30.2
- net SWCLK: now also U5.37 (PA14)
- net SWDIO: now also U5.34 (PA13)
- net V_FB: now also U5.11 (PA1), R19.1
- net at C20.1, C21.1, L3.2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: now also J3.1 (Pin_1)
- net at C20.2, C21.2, R12.1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: now also J3.2 (Pin_2)
- net ENC_A: now reaches SW1.A
- net ENC_A: now also U5.18 (PB0)
- net ENC_B: now reaches SW1.B
- net ENC_B: now also U5.46 (PB9)
- net SCL: now reaches U5.21 (PB10)
- net SDA: now reaches U5.22 (PB11)
- net V_PWM: now reaches U5.29 (PA8)
- net at U5.44 (BOOT0): now also R17.1
- no-connect marks 0 -> 26
Other:
- note added: "Vin: 12V-48V"
- note added: "Vout: 0.2V-32V"
- note removed: "Vin: 12V-50V"
- note removed: "Vout: 0.2V-48V"
- moved on the sheet: C1, C10, C11, C12, C13, C14, C15, C16, C17, C18, C19, C2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

Commit message: Place component on board
Parts:
- removed C1: C0603/1nF, Capacitor_SMD:C_0603_1608Metric, symbol Device:C
- removed D1: 1N5819, Diode_THT:D_DO-41_SOD81_P10.16mm_Horizontal, symbol Diode:1N5819
- added C1, C36: Cp/680uF/63V, Capacitor_THT:CP_Radial_D13.0mm_P5.00mm, symbol Device:C_Polarized
- added C32, C33, C34, C35: C0603/20pF, Capacitor_SMD:C_0603_1608Metric, symbol Device:C
- added D1: SS24, Diode_SMD:D_SMA, symbol Diode:SS34
- added D4: 1N4148W, Diode_SMD:D_SOD-123, symbol Diode:1N4148
- added F1: Fuse, Fuse:Fuse_Blade_Mini_directSolder, symbol Device:Fuse
- added J5: FAN, Connector_JST:JST_XH_B2B-XH-A_1x02_P2.50mm_Vertical, symbol Connector:Conn_01x02_Pin
- added Q1: 2N7002, Package_TO_SOT_SMD:SOT-23, symbol Transistor_FET:2N7002
- added R20: R0603/10k, Resistor_SMD:R_0603_1608Metric, symbol Device:R
- added R21: R2512/0.002R/3W, Resistor_SMD:R_2512_6332Metric, symbol Device:R
- added R22, R23, R24, R25: R0603/10K, Resistor_SMD:R_0603_1608Metric, symbol Device:R
- added Y1: 8Mhz, Crystal:Crystal_SMD_5032-2Pin_5.0x3.2mm, symbol Device:Crystal
- added Y2: 32.768K, Crystal:Crystal_SMD_3215-2Pin_3.2x1.5mm, symbol Device:Crystal
- C10, C13, C14: footprint Capacitor_SMD:C_0603_1608Metric -> Capacitor_SMD:C_0805_2012Metric
- C11, C22, C23: value Cp/470uF/63V -> Cp/680uF/63V; footprint Capacitor_THT:CP_Radial_D12.5mm_P5.00mm -> Capacitor_THT:CP_Radial_D13.0mm_P5.00mm
- C18: value C0603/68pF -> C0603/150pF
- C20: value 220uF/65V -> Cp/680uF/63V; footprint Connector_JST:JST_XH_B5B-XH-AM_1x05_P2.50mm_Vertical -> Capacitor_THT:CP_Radial_D13.0mm_P5.00mm
- C21: value C0603/100nF -> C0603/100nF/50V
- D3: value SS34 -> SS24
- D8: value 1N4148 -> 1N4148W; footprint Diode_THT:D_DO-35_SOD27_P7.62mm_Horizontal -> Diode_SMD:D_SOD-123
- D9: footprint Diode_THT:D_DO-35_SOD27_P7.62mm_Horizontal -> Diode_SMD:D_SOD-123
- J1: value Conn_01x05_Pin -> DEBUG
- J2, J3: footprint TerminalBlock_Phoenix:TerminalBlock_Phoenix_MKDS-1,5-2-5.08_1x02_P5.08mm_Horizontal -> TerminalBlock_Dinkle:TerminalBlock_Dinkle_DT-55-B01X-02_P10.00mm
- J4: value Conn_01x04_Pin -> LCD
- L1: value L/47uH /620mA -> L/47uH/620mA
- L2: footprint (none) -> Inductor_SMD:L_APV_APH0412
- L3: value 47uF/25A -> 68uF/25A; footprint (none) -> Programmable_Buck:Inductor_36x23x15MM
- R12, R13, R15: value R0603/150K -> R0603/1K
- R14: value R0603/150K -> R0603/75K
- R41: value R0603/150K -> R0603/100K
- R53: value RS/0.002R -> R2512/0.002R/3W; footprint Resistor_SMD:R_0603_1608Metric -> Resistor_SMD:R_2512_6332Metric
- U4: footprint Package_SO:SOIC-16_3.9x9.9mm_P1.27mm -> Package_SO:SOP-16_4.4x10.4mm_P1.27mm
- U6: footprint Package_DIP:CERDIP-8_W7.62mm_SideBrazed_LongPads_Socket -> Package_SO:SOIC-8_3.9x4.9mm_P1.27mm
Connections:
- net I2C0_SCL is gone; now on net SCL: J4.3 (Pin_3)
- net I2C0_SDA is gone; now on net SDA: J4.4 (Pin_4)
- net +12V: now also D1.2 (A), D4.1 (K), J5.1 (Pin_1)
- net +3.3V: now also R22.1, R23.1
- net ENC_BUTTON: now also C5.1
- net GND: now also C32.2, C33.2, C34.2, C35.2, Q1.2 (S), R21.1, R24.2; no longer C5.1
- net SCL: now also R22.2
- net SDA: now also R23.2
- net V_FB: now also R20.1; no longer R52.1, U5.11 (PA1)
- net at C20.1, C21.1, L3.2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: now also C1.1, C36.1, F1.1; no longer J3.1 (Pin_1)
- net at C20.2, C21.2, J3.2 (Pin_2)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: now also C1.2, C36.2, R21.2
- net at C19.1, U6.8 (VB): now also D1.1 (K)
- net FAN_ON: now reaches U5.2 (PC13)
- net FAN_ON: now also R25.1
- net at U5.3 (PC14): now also C34.1, Y2.2
- net at U5.4 (PC15): now also C35.1, Y2.1
- net at U5.5 (PD0): now also C32.1, Y1.2
- net at U5.6 (PD1): now also C33.1, Y1.1
- new net: D4.2 (A), J5.2 (Pin_2), Q1.3 (D)
- new net: Q1.1 (G), R24.1, R25.2
- new net: F1.2, J3.1 (Pin_1)
- new net V_fb: R20.2, R52.1, U5.11 (PA1)
- no-connect marks 26 -> 20
Other:
- note added: "66kHz"
- note removed: "75kHz"
- moved on the sheet: C11, C12, C13, C14, C15, C16, C17, C18, C19, C2, C21, C22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

Commit message: Finalize PCb
Connections:
- net FAN_ON: now also U5.38 (PA15); no longer U5.2 (PC13)
- no-connect marks 20 -> 19
Changed lines of the file:
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@@
 	)
 	(no_connect
-		(at 289.56 226.06)
-	)
-	(no_connect
 		(at 289.56 195.58)
 	)
@@
 	(wire
 		(pts
+			(xy 289.56 226.06) (xy 306.07 226.06)
+		)
+		(stroke
+			(width 0)
+			(type default)
+		)
+	)
+	(wire
+		(pts
 			(xy 45.72 97.79) (xy 64.77 97.79)
 		)
@@
 	(wire
 		(pts
-			(xy 254 205.74) (xy 245.11 205.74)
-		)
-		(stroke
-			(width 0)
-			(type default)
-		)
-	)
-	(wire
-		(pts
 			(xy 35.56 189.23) (xy 33.02 189.23)
 		)
@@
 		)
 	)
-	(label "FAN_ON"
-		(at 245.11 205.74 0)
-		(effects
-			(font
-				(size 1.27 1.27)
-			)
-			(justify left bottom)
-		)
-	)
 	(label "SWCLK"
 		(at 306.07 223.52 180)
@@
 		(effects
 			(font
+				(size 1.27 1.27)
+			)
+			(justify right bottom)
+		)
+	)
+	(label "FAN_ON"
+		(at 306.07 226.06 180)
+		(effects
+			(font
